File: Schematics/CAN-Transciever.kicad_sch (KiCad schematic)
At the start: 6 parts, among them U1 SN65HVD230

Commit message: clean up of routing
Parts:
- JP1: LCSC (none) -> C474893
Changed lines of the file:
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@@
+			)
+		)
+		(property "LCSC" "C474893"
+			(at 153.67 95.25 0)
+			(effects
+				(font
+					(size 1.27 1.27)
+				)
+				(hide yes)
 			)
 		)
